File: bed_face-pcb.kicad_pcb (KiCad board)
At the start: 2 copper layers, 228.6 x 76.2 mm, 106 parts, among them SW1 SW_Push, U1 ProMicro

Commit message: improved GND fill after encoder placement/tracks
Routing:
- net GND: track 27.3 -> 36.3 mm, vias 23 -> 32
Changed lines of the file:
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@@
     (thickness 1.6)
     (drawings 8)
-    (tracks 570)
+    (tracks 583)
     (zones 0)
     (modules 106)
@@
   (segment (start 242.00125 70.32625) (end 243.18125 71.50625) (width 0.25) (layer B.Cu) (net 14))
   (segment (start 237.49 70.32625) (end 242.00125 70.32625) (width 0.25) (layer B.Cu) (net 14))
-  (segment (start 261.07 70.32625) (end 262.25 71.50625) (width 0.25) (layer B.Cu) (net 67))
-  (segment (start 256.54 70.32625) (end 261.07 70.32625) (width 0.25) (layer B.Cu) (net 67))
   (segment (start 73.812501 91.356249) (end 74.6125 90.55625) (width 0.25) (layer B.Cu) (net 15))
   (segment (start 73.352449 91.816301) (end 73.812501 91.356249) (width 0.25) (layer B.Cu) (net 15))
@@
   (segment (start 242.00125 89.37625) (end 243.18125 90.55625) (width 0.25) (layer B.Cu) (net 24))
   (segment (start 237.49 89.37625) (end 242.00125 89.37625) (width 0.25) (layer B.Cu) (net 24))
-  (segment (start 261.05125 89.37625) (end 262.23125 90.55625) (width 0.25) (layer B.Cu) (net 68))
-  (segment (start 256.54 89.37625) (end 261.05125 89.37625) (width 0.25) (layer B.Cu) (net 68))
   (segment (start 70.4825 108.42625) (end 71.73125 109.675) (width 0.25) (layer B.Cu) (net 25))
   (segment (start 66.04 108.42625) (end 70.4825 108.42625) (width 0.25) (layer B.Cu) (net 25))
@@
   (segment (start 242.00125 108.42625) (end 243.18125 109.60625) (width 0.25) (layer B.Cu) (net 34))
   (segment (start 237.49 108.42625) (end 242.00125 108.42625) (width 0.25) (layer B.Cu) (net 34))
-  (segment (start 261.05125 108.42625) (end 262.23125 109.60625) (width 0.25) (layer B.Cu) (net 69))
-  (segment (start 256.54 108.42625) (end 261.05125 108.42625) (width 0.25) (layer B.Cu) (net 69))
   (segment (start 70.55125 127.47625) (end 71.73125 128.65625) (width 0.25) (layer B.Cu) (net 35))
   (segment (start 66.04 127.47625) (end 70.55125 127.47625) (width 0.25) (layer B.Cu) (net 35))
@@
   (segment (start 242.00125 127.47625) (end 243.18125 128.65625) (width 0.25) (layer B.Cu) (net 44))
   (segment (start 237.49 127.47625) (end 242.00125 127.47625) (width 0.25) (layer B.Cu) (net 44))
-  (segment (start 261.05125 127.47625) (end 262.23125 128.65625) (width 0.25) (layer B.Cu) (net 70))
-  (segment (start 256.54 127.47625) (end 261.05125 127.47625) (width 0.25) (layer B.Cu) (net 70))
   (segment (start 40.64 69.71625) (end 40.64 72.86625) (width 0.25) (layer F.Cu) (net 45))
   (segment (start 41.95 68.40625) (end 40.64 69.71625) (width 0.25) (layer F.Cu) (net 45))
@@
   (via (at 62.5 89.5) (size 0.8) (drill 0.4) (layers F.Cu B.Cu) (net 57))
   (via (at 63.5 82.5) (size 0.8) (drill 0.4) (layers F.Cu B.Cu) (net 57))
-  (via (at 82.5 81.5) (size 0.8) (drill 0.4) (layers F.Cu B.Cu) (net 57))
   (via (at 82 89.5) (size 0.8) (drill 0.4) (layers F.Cu B.Cu) (net 57))
   (via (at 68.5 90) (size 0.8) (drill 0.4) (layers F.Cu B.Cu) (net 57))
@@
   (segment (start 254 140.05625) (end 254 138.90625) (width 0.381) (layer F.Cu) (net 57))
   (segment (start 254 138.90625) (end 254.79375 138.1125) (width 0.381) (layer F.Cu) (net 57))
+  (via (at 188.9125 113.50625) (size 0.8) (drill 0.4) (layers F.Cu B.Cu) (net 57))
+  (via (at 208.75625 127.79375) (size 0.8) (drill 0.4) (layers F.Cu B.Cu) (net 57))
+  (via (at 169.8625 113.50625) (size 0.8) (drill 0.4) (layers F.Cu B.Cu) (net 57))
+  (via (at 150.8125 113.50625) (size 0.8) (drill 0.4) (layers F.Cu B.Cu) (net 57))
+  (via (at 207.9625 113.50625) (size 0.8) (drill 0.4) (layers F.Cu B.Cu) (net 57))
+  (via (at 209.55 86.51875) (size 0.8) (drill 0.4) (layers F.Cu B.Cu) (net 57))
+  (via (at 92.86875 81.75625) (size 0.8) (drill 0.4) (layers F.Cu B.Cu) (net 57))
+  (via (at 96.04375 80.049999) (size 0.8) (drill 0.4) (layers F.Cu B.Cu) (net 57))
+  (segment (start 92.86875 81.75625) (end 94.337499 81.75625) (width 0.381) (layer F.Cu) (net 57))
+  (segment (start 94.337499 81.75625) (end 96.04375 80.049999) (width 0.381) (layer F.Cu) (net 57))
+  (via (at 100.80625 80.9625) (size 0.8) (drill 0.4) (layers F.Cu B.Cu) (net 57))
+  (segment (start 96.04375 80.049999) (end 99.893749 80.049999) (width 0.381) (layer B.Cu) (net 57))
+  (segment (start 99.893749 80.049999) (end 100.80625 80.9625) (width 0.381) (layer B.Cu) (net 57))
+  (via (at 75.40625 82.55) (size 0.8) (drill 0.4) (layers F.Cu B.Cu) (net 57))
   (segment (start 208.3 69.8) (end 207 71.1) (width 0.25) (layer F.Cu) (net 58))
   (segment (start 207 71.1) (end 207 80) (width 0.25) (layer F.Cu) (net 58))
@@
   (segment (start 204.64632 82.38493) (end 207 80.03125) (width 0.25) (layer B.Cu) (net 58))
   (segment (start 71.12 80.455) (end 71.455 80.455) (width 0.25) (layer B.Cu) (net 60))
-  (segment (start 55.88 80.455) (end 55.545 80.455) (width 0.25) (layer F.Cu) (net 61))
-  (segment (start 72.321301 83.234881) (end 73.27139 84.18497) (width 0.25) (layer B.Cu) (net 61))
-  (segment (start 72.321301 82.418375) (end 72.321301 83.234881) (width 0.25) (layer B.Cu) (net 61))
-  (segment (start 71.559227 81.656301) (end 72.321301 82.418375) (width 0.25) (layer B.Cu) (net 61))
-  (segment (start 70.543375 81.656301) (end 71.559227 81.656301) (width 0.25) (layer B.Cu) (net 61))
-  (segment (start 55.88 80.455) (end 69.342074 80.455) (width 0.25) (layer B.Cu) (net 61))
-  (segment (start 69.342074 80.455) (end 70.543375 81.656301) (width 0.25) (layer B.Cu) (net 61))
-  (segment (start 73.27139 84.18497) (end 223.40872 84.18497) (width 0.25) (layer B.Cu) (net 61))
   (segment (start 71.12 80.580664) (end 72.771311 82.231975) (width 0.25) (layer B.Cu) (net 60))
   (segment (start 71.12 80.455) (end 71.12 80.580664) (width 0.25) (layer B.Cu) (net 60))
@@
   (segment (start 256.5 123.595248) (end 255.089999 125.005249) (width 0.25) (layer F.Cu) (net 60))
   (segment (start 256.5 121.00625) (end 256.5 123.595248) (width 0.25) (layer F.Cu) (net 60))
+  (segment (start 55.88 80.455) (end 55.545 80.455) (width 0.25) (layer F.Cu) (net 61))
+  (segment (start 72.321301 83.234881) (end 73.27139 84.18497) (width 0.25) (layer B.Cu) (net 61))
+  (segment (start 72.321301 82.418375) (end 72.321301 83.234881) (width 0.25) (layer B.Cu) (net 61))
+  (segment (start 71.559227 81.656301) (end 72.321301 82.418375) (width 0.25) (layer B.Cu) (net 61))
+  (segment (start 70.543375 81.656301) (end 71.559227 81.656301) (width 0.25) (layer B.Cu) (net 61))
+  (segment (start 55.88 80.455) (end 69.342074 80.455) (width 0.25) (layer B.Cu) (net 61))
+  (segment (start 69.342074 80.455) (end 70.543375 81.656301) (width 0.25) (layer B.Cu) (net 61))
+  (segment (start 73.27139 84.18497) (end 223.40872 84.18497) (width 0.25) (layer B.Cu) (net 61))
   (segment (start 250.22128 84.18497) (end 223.40872 84.18497) (width 0.25) (layer B.Cu) (net 61))
   (segment (start 251.5 82.90625) (end 250.22128 84.18497) (width 0.25) (layer B.Cu) (net 61))
@@
   (segment (start 226.2875 98.35625) (end 219.86875 104.775) (width 0.25) (layer F.Cu) (net 66))
   (segment (start 243.18125 98.35625) (end 226.2875 98.35625) (width 0.25) (layer F.Cu) (net 66))
+  (segment (start 261.07 70.32625) (end 262.25 71.50625) (width 0.25) (layer B.Cu) (net 67))
+  (segment (start 256.54 70.32625) (end 261.07 70.32625) (width 0.25) (layer B.Cu) (net 67))
   (segment (start 256.5 70.28625) (end 256.54 70.32625) (width 0.25) (layer F.Cu) (net 67))
   (segment (start 256.5 68.40625) (end 256.5 70.28625) (width 0.25) (layer F.Cu) (net 67))
+  (segment (start 261.05125 89.37625) (end 262.23125 90.55625) (width 0.25) (layer B.Cu) (net 68))
+  (segment (start 256.54 89.37625) (end 261.05125 89.37625) (width 0.25) (layer B.Cu) (net 68))
   (segment (start 256.5 89.33625) (end 256.54 89.37625) (width 0.25) (layer F.Cu) (net 68))
   (segment (start 256.5 87.45625) (end 256.5 89.33625) (width 0.25) (layer F.Cu) (net 68))
+  (segment (start 261.05125 108.42625) (end 262.23125 109.60625) (width 0.25) (layer B.Cu) (net 69))
+  (segment (start 256.54 108.42625) (end 261.05125 108.42625) (width 0.25) (layer B.Cu) (net 69))
   (segment (start 256.5 108.38625) (end 256.54 108.42625) (width 0.25) (layer F.Cu) (net 69))
   (segment (start 256.5 106.50625) (end 256.5 108.38625) (width 0.25) (layer F.Cu) (net 69))
+  (segment (start 261.05125 127.47625) (end 262.23125 128.65625) (width 0.25) (layer B.Cu) (net 70))
+  (segment (start 256.54 127.47625) (end 261.05125 127.47625) (width 0.25) (layer B.Cu) (net 70))
   (segment (start 256.5 127.43625) (end 256.54 127.47625) (width 0.25) (layer F.Cu) (net 70))
   (segment (start 256.5 125.55625) (end 256.5 127.43625) (width 0.25) (layer F.Cu) (net 70))
